Commit message: commit rsv10 launchs

File: akagachi_demo/model/rsv10_eyes.urdf.xacro (robot description, xacro)
@@ -33,5 +33,5 @@
     <visual>
       <geometry>
-        <mesh filename="package://blink_robot/mesh/1B_eyelid.stl"/>
+        <mesh scale="0.0013 0.0013 0.0013"  filename="package://blink_robot/mesh/1B_eyelid.stl"/>
       </geometry>
       <material name="blue">
@@ -70,5 +70,5 @@
     <parent link="eye_r"/>
     <child link="eyelid"/>
-    <origin xyz="0 -0.05 0"/>
+    <origin xyz="0 0 0"/>
     <axis xyz="0 0 1"/>
     <limit lower="${-40*deg2rad}" upper="${40*deg2rad}" effort="1" velocity="1"/>

Commit message: update syncronized  blinking function

File: akagachi_demo/model/rsv10_eyes.urdf.xacro (robot description, xacro)
@@ -33,5 +33,5 @@
     <visual>
       <geometry>
-        <mesh scale="0.0013 0.0013 0.0013"  filename="package://blink_robot/mesh/1B_eyelid.stl"/>
+        <mesh scale="0.0013 0.0013 0.0013"  filename="package://akagachi_demo/model/1B_eyelid.stl"/>
       </geometry>
       <material name="blue">
@@ -70,6 +70,6 @@
     <parent link="eye_r"/>
     <child link="eyelid"/>
-    <origin xyz="0 0 0"/>
-    <axis xyz="0 0 1"/>
+    <origin xyz="0 0 0" rpy="4.8 3.14 -1.7"/>
+    <axis xyz="-1 0 0"/>
     <limit lower="${-40*deg2rad}" upper="${40*deg2rad}" effort="1" velocity="1"/>
   </joint>
